File: Daylight_on_a_Stick/Daylight/Daylight.kicad_pcb (KiCad board)
At the start: 2 copper layers, 270 x 11 mm, 33 parts, among them J1 Conn_01x02, J2 Conn_01x02

Commit message: Fixed some Layout LED footprint issues
Other:
- board text added: "Daylight on a stick by Blamm Daybreak by Vector 3D V2.1"
- board text removed: "Daylight on a stick by Blamm Daybreak by Vector 3D V2"
Changed lines of the file:
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@@
     (effects (font (size 1.5 1.5) (thickness 0.25)) (justify right mirror))
   )
-  (gr_text "Daylight on a stick by Blamm\nDaybreak by Vector 3D\nV2" (at 147.5 33) (layer "B.SilkS")
+  (gr_text "Daylight on a stick by Blamm\nDaybreak by Vector 3D\nV2.1" (at 147.5 33) (layer "B.SilkS")
     (effects (font (size 1 1) (thickness 0.15)) (justify mirror))
   )
@@
     (connect_pads (clearance 0.508))
     (min_thickness 0.254) (filled_areas_thickness no)
-    (fill yes (thermal_gap 0.508) (thermal_bridge_width 0.508))
+    (fill yes (thermal_gap 0.5) (thermal_bridge_width 0.5))
     (polygon
       (pts
@@
     (connect_pads (clearance 0.508))
     (min_thickness 0.254) (filled_areas_thickness no)
-    (fill yes (thermal_gap 0) (thermal_bridge_width 0.508))
+    (fill yes (thermal_gap 0.5) (thermal_bridge_width 0.5))
     (polygon
       (pts
@@
     (connect_pads (clearance 0.508))
     (min_thickness 0.254) (filled_areas_thickness no)
-    (fill yes (thermal_gap 0.508) (thermal_bridge_width 0.8))
+    (fill yes (thermal_gap 0.5) (thermal_bridge_width 0.5))
     (polygon
       (pts

Commit message: Daylight (all) V2.2
The JST XH silkscreen did not match the connectors very well so it has been adjusted.
Added small front silkscreen to indicate pins
Adjusted one connector on day_mini that was misplaced 1mm.
Parts:
- J1, J2: footprint Connector_JST:JST_XH_S2B-XH-A_1x02_P2.50mm_Horizontal -> Daylight:JST_XH_S2B-XH-A_1x02_P2.50mm_Horizontal Daylight
Routing:
- net GND: vias 49 -> 48
Other:
- board text added: "+ -"
- board text added: "- +"
- board text added: "Daylight on a stick by Blamm Daybreak by Vector 3D V2.2"
- board text removed: "Daylight on a stick by Blamm Daybreak by Vector 3D V2.1"
