File: Daylight_on_a_Stick/Daylight/Daylight.kicad_pcb (KiCad board)
At the start: 2 copper layers, 270 x 11 mm, 56 parts, among them J1 Conn_01x02, J2 Conn_01x02

Commit message: Minor LED Updates
Parts:
- removed the REF** at (58.1, 38.1)
- removed the REF** at (108.1, 38.1)
- removed the REF** at (283.1, 32.6)
- removed the REF** at (160.1, 38.1)
- removed the REF** at (237.1, 38.1)
- removed the REF** at (108.1, 27.1)
- removed the REF** at (186.1, 38.1)
- removed the REF** at (211.1, 38.1)
- removed the REF** at (58.1, 27.1)
- removed the REF** at (160.1, 27.1)
- removed the REF** at (237.1, 27.1)
- removed the REF** at (186.1, 27.1)
- removed the REF** at (211.1, 27.1)
- removed the REF** at (13.1, 32.6)
- moved REF** 56.0 mm to (190.1, 27.1)
- moved REF** 56.0 mm to (190.1, 38.1)
- moved REF** 34.5 mm to (117.6, 27.1)
- moved REF** 34.5 mm to (117.6, 38.1)
- moved REF** 12.0 mm to (45.1, 38.1)
- moved REF** 12.0 mm to (45.1, 27.1)
- moved REF** 12.0 mm to (251.1, 27.1)
- moved REF** 12.0 mm to (251.1, 38.1)
