File: Daylight_on_a_Stick/Daylight/Daylight.kicad_sch (KiCad schematic)
At the start: 31 parts

Commit message: Daylight (all) V2.2
The JST XH silkscreen did not match the connectors very well so it has been adjusted.
Added small front silkscreen to indicate pins
Adjusted one connector on day_mini that was misplaced 1mm.
Parts:
- D1, D10, D11, D12, D13, D14, D15, D16, D17, D18, D19, D2, D20, D21, D3, D4, D5, D6, D7, D8, D9: value (none) -> LED_ALT; footprint (none) -> LED_SMD:LED_PLCC_2835
- H1, H2: value (none) -> MountingHole; footprint (none) -> MountingHole:MountingHole_3.2mm_M3_Pad_Via
- J1, J2: value (none) -> Conn_01x02; footprint (none) -> Connector_JST:JST_XH_S2B-XH-A_1x02_P2.50mm_Horizontal
- R1, R2, R3, R4, R5, R6: value (none) -> 20R 0.25W; footprint (none) -> Resistor_SMD:R_1206_3216Metric
