File: Daylight_on_a_Stick/Daylight/Daylight.kicad_sch (KiCad schematic)
At the start: 31 parts, among them J1 Conn_01x02, J2 Conn_01x02

Commit message: Minor LED Updates
Parts:
- J1, J2: LCSC (none) -> C2908611; now in the parts list
Changed lines of the file:
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@@
   )
   (symbol (lib_id "Connector_Generic:Conn_01x02") (at 80.01 77.47 0) (mirror y) (unit 1)
-    (in_bom no) (on_board yes) (fields_autoplaced)
+    (in_bom yes) (on_board yes) (fields_autoplaced)
     (property "Reference" "J1" (id 0) (at 80.01 71.12 0))
     (property "Value" "Conn_01x02" (id 1) (at 80.01 73.66 0))
@@
       (effects (font (size 1.27 1.27)) hide)
     )
+    (property "LCSC" "C2908611" (id 4) (at 80.01 77.47 0)
+      (effects (font (size 1.27 1.27)) hide)
+    )
     (pin "1")
     (pin "2")
@@
   )
   (symbol (lib_id "Connector_Generic:Conn_01x02") (at 62.23 77.47 0) (unit 1)
-    (in_bom no) (on_board yes)
+    (in_bom yes) (on_board yes)
     (property "Reference" "J2" (id 0) (at 62.23 71.12 0)
       (effects (font (size 1.27 1.27)) (justify left))
@@
       (effects (font (size 1.27 1.27)) hide)
     )
+    (property "LCSC" "C2908611" (id 4) (at 62.23 77.47 0)
+      (effects (font (size 1.27 1.27)) hide)
+    )
