File: Daylight_on_a_Stick/Daylight_UV/Daylight_UV.kicad_pcb (KiCad board)
At the start: 2 copper layers, 270 x 11 mm, 56 parts, among them J1 Conn_01x02, J2 Conn_01x02

Commit message: Minor Updates
Parts:
- removed the G*** at (201.0, 32.5)
Other:
- board text added: "Daylight on a stick by Blamm Daybreak UV by Vector 3D V1.0"
- board text added: "This product uses 365nm UV LEDs. Be sure to take appropriate precautions."
- board text added: "WARNING"
- board text removed: "Daylight on a stick by Blamm Daybreak by Vector 3D V2.3"
