File: Daylight_on_a_Stick/Daylight_UV/Daylight_UV.kicad_sch (KiCad schematic)
At the start: 31 parts, among them J1 Conn_01x02, J2 Conn_01x02

Commit message: Minor Updates
Parts:
- D1, D10, D11, D12, D13, D14, D15, D16, D17, D18, D19, D2, D20, D21, D3, D4, D5, D6, D7, D8, D9: value LED_ALT -> LED_UV; LCSC C2843876 -> C2915615; ManfNum XL-2835UWC-02 -> (none); abv.Footprint 2835 -> (none)
- R1, R2, R3, R4, R5, R6: ManfNum 1206W4F200JT5E -> (none); abv.Footprint 1206 -> (none)
Other:
- note added: "UV LED 3.2v 150ma"
- note removed: "3.2v"
