File: Daylight_on_a_Stick/Daylight_UV_Mini/Daylight_UV_Mini.kicad_pcb (KiCad board)
At the start: 2 copper layers, 170 x 11 mm, 25 parts, among them J1 Conn_01x02, J2 Conn_01x02

Commit message: Minor Updates
Parts:
- removed the G*** at (130.7, 33.0)
Other:
- board text added: "Daylight on a stick by Blamm Daybreak UV Mini by Vector 3D V1.0"
- board text added: "This product uses 365nm UV LEDs. Be sure to take precautions and use appropriate safety equipment."
- board text added: "WARNING"
- board text removed: "Daylight on a stick by Blamm Daybreak Mini by Vector 3D V2.3"
