File: Daylight_on_a_Stick/Daylight_UV_Mini/Daylight_UV_Mini.kicad_sch (KiCad schematic)
At the start: 31 parts, among them J1 Conn_01x02, J2 Conn_01x02

Commit message: Minor Updates
Parts:
- removed D13, D14, D15, D16, D17, D18, D21: LED_ALT, LED_SMD:LED_PLCC_2835, symbol Device:LED_ALT
- removed R5, R6: 20R 0.25W, Resistor_SMD:R_1206_3216Metric, symbol Device:R_Small
- D1, D2, D3, D4, D5, D6: value LED_ALT -> LED_UV; LCSC C2843876 -> C2915615; ManfNum XL-2835UWC-02 -> (none); abv.Footprint 2835 -> (none)
- D10: renamed from D9; value LED_ALT -> LED_UV; LCSC C2843876 -> C2915615; ManfNum XL-2835UWC-02 -> (none); abv.Footprint 2835 -> (none)
- D11: renamed from D10; value LED_ALT -> LED_UV; LCSC C2843876 -> C2915615; ManfNum XL-2835UWC-02 -> (none); abv.Footprint 2835 -> (none)
- D12: renamed from D11; value LED_ALT -> LED_UV; LCSC C2843876 -> C2915615; ManfNum XL-2835UWC-02 -> (none); abv.Footprint 2835 -> (none)
- D13: renamed from D12; value LED_ALT -> LED_UV; LCSC C2843876 -> C2915615; ManfNum XL-2835UWC-02 -> (none); abv.Footprint 2835 -> (none)
- D14: renamed from D20; value LED_ALT -> LED_UV; LCSC C2843876 -> C2915615; ManfNum XL-2835UWC-02 -> (none); abv.Footprint 2835 -> (none)
- D7: renamed from D19; value LED_ALT -> LED_UV; LCSC C2843876 -> C2915615; ManfNum XL-2835UWC-02 -> (none); abv.Footprint 2835 -> (none)
- D8: renamed from D7; value LED_ALT -> LED_UV; LCSC C2843876 -> C2915615; ManfNum XL-2835UWC-02 -> (none); abv.Footprint 2835 -> (none)
- D9: renamed from D8; value LED_ALT -> LED_UV; LCSC C2843876 -> C2915615; ManfNum XL-2835UWC-02 -> (none); abv.Footprint 2835 -> (none)
- R1, R2, R3, R4: ManfNum 1206W4F200JT5E -> (none); abv.Footprint 1206 -> (none)
- renumbered J2 to J1, J1 to J2
Other:
- note added: "UV LED 3.2v 150ma"
- note removed: "3.2v"
