File: Daylight_on_a_Stick/Daylight_Mini/Daylight_mini.kicad_pcb (KiCad board)
At the start: 2 copper layers, 170 x 11 mm, 25 parts, among them J1 Conn_01x02, J2 Conn_01x02

Commit message: Minor LED Updates
Parts:
- added REF**: Tab, kikit:Tab, F.Cu at (35.0, 38.5)
- added REF**: Tab, kikit:Tab, F.Cu at (98.0, 27.5)
- added REF**: Tab, kikit:Tab, F.Cu at (35.0, 27.5)
- added REF**: Tab, kikit:Tab, F.Cu at (98.0, 38.5)
- added REF**: Tab, kikit:Tab, F.Cu at (161.0, 38.5)
- added REF**: Tab, kikit:Tab, F.Cu at (161.0, 27.5)
Other:
- board text added: "Daylight on a stick by Blamm Daybreak Mini by Vector 3D V2.4"
- board text removed: "Daylight on a stick by Blamm Daybreak Mini by Vector 3D V2.3"
