File: Daylight_on_a_Stick/Daylight_Neo/Daylight_Neo.kicad_pcb (KiCad board)
At the start: 2 copper layers, 270 x 11 mm, 32 parts, among them J1 IN, J2 OUT

Commit message: Fixed some Layout LED footprint issues
Parts:
- D1, D10, D11, D12, D13, D2, D3, D4, D5, D6, D7, D8, D9: footprint LED_SMD:LED_SK6812MINI_PLCC4_3.5x3.5mm_P1.75mm -> Daylight:XL-3528RGBW-WS2812B
- moved C2 0.90 mm to (56.4, 33.0)
- turned D1 to 90 degrees
- turned D10 to 90 degrees
- turned D11 to 90 degrees
- turned D12 to 90 degrees
- turned D13 to 90 degrees
- turned D2 to 90 degrees
- turned D3 to 90 degrees
- turned D4 to 90 degrees
- turned D5 to 90 degrees
- turned D6 to 90 degrees
- turned D7 to 90 degrees
- turned D8 to 90 degrees
- turned D9 to 90 degrees
Connections:
- D1 pad 1: Net-(D1-Pad1) -> GND
- D1 pad 2: GND -> Dstart
- D1 pad 3: Dstart -> +5V
- D1 pad 4: +5V -> Net-(D1-Pad4)
- D10 pad 1: Net-(D10-Pad1) -> GND
- D10 pad 2: GND -> Net-(D10-Pad2)
- D10 pad 3: Net-(D10-Pad3) -> +5V
- D10 pad 4: +5V -> Net-(D10-Pad4)
- D11 pad 1: Net-(D11-Pad1) -> GND
- D11 pad 2: GND -> Net-(D10-Pad4)
- D11 pad 3: Net-(D10-Pad1) -> +5V
- D11 pad 4: +5V -> Net-(D11-Pad4)
- D12 pad 1: Net-(D12-Pad1) -> GND
- D12 pad 2: GND -> Net-(D11-Pad4)
- D12 pad 3: Net-(D11-Pad1) -> +5V
- D12 pad 4: +5V -> Net-(D12-Pad4)
- D13 pad 1: Dend -> GND
- D13 pad 2: GND -> Net-(D12-Pad4)
- D13 pad 3: Net-(D12-Pad1) -> +5V
- D13 pad 4: +5V -> Dend
- D2 pad 1: Net-(D2-Pad1) -> GND
- D2 pad 2: GND -> Net-(D1-Pad4)
- D2 pad 3: Net-(D1-Pad1) -> +5V
- D2 pad 4: +5V -> Net-(D2-Pad4)
- D3 pad 1: Net-(D3-Pad1) -> GND
- D3 pad 2: GND -> Net-(D2-Pad4)
- D3 pad 3: Net-(D2-Pad1) -> +5V
- D3 pad 4: +5V -> Net-(D3-Pad4)
- D4 pad 1: Net-(D4-Pad1) -> GND
- D4 pad 2: GND -> Net-(D3-Pad4)
- D4 pad 3: Net-(D3-Pad1) -> +5V
- D4 pad 4: +5V -> Net-(D4-Pad4)
- D5 pad 1: Net-(D5-Pad1) -> GND
- D5 pad 2: GND -> Net-(D4-Pad4)
- D5 pad 3: Net-(D4-Pad1) -> +5V
- D5 pad 4: +5V -> Net-(D5-Pad4)
- D6 pad 1: Net-(D6-Pad1) -> GND
- D6 pad 2: GND -> Net-(D5-Pad4)
- D6 pad 3: Net-(D5-Pad1) -> +5V
- D6 pad 4: +5V -> Net-(D6-Pad4)
- D7 pad 1: Net-(D7-Pad1) -> GND
- D7 pad 2: GND -> Net-(D6-Pad4)
- D7 pad 3: Net-(D6-Pad1) -> +5V
- D7 pad 4: +5V -> Net-(D7-Pad4)
- D8 pad 1: Net-(D8-Pad1) -> GND
- D8 pad 2: GND -> Net-(D7-Pad4)
- D8 pad 3: Net-(D7-Pad1) -> +5V
- D8 pad 4: +5V -> Net-(D8-Pad4)
- D9 pad 1: Net-(D10-Pad3) -> GND
- D9 pad 2: GND -> Net-(D8-Pad4)
- D9 pad 3: Net-(D8-Pad1) -> +5V
- D9 pad 4: +5V -> Net-(D10-Pad2)
Routing:
- net Net-(D12-Pad4): track 0.00 -> 21.6 mm
- net Net-(D1-Pad4): track 0.00 -> 20.6 mm
- net Net-(D12-Pad1): track 19.5 -> 0.00 mm
- net Net-(D5-Pad4): track 0.00 -> 18.6 mm
- net Net-(D2-Pad4): track 0.00 -> 18.6 mm
- net Net-(D10-Pad2): track 0.00 -> 18.6 mm
- net Net-(D4-Pad4): track 0.00 -> 18.6 mm
- net Net-(D3-Pad4): track 0.00 -> 18.6 mm
- net Net-(D8-Pad4): track 0.00 -> 18.6 mm
- net Net-(D7-Pad4): track 0.00 -> 18.6 mm
- net Net-(D6-Pad4): track 0.00 -> 18.6 mm
- net Net-(D11-Pad4): track 0.00 -> 18.6 mm
- net Net-(D10-Pad4): track 0.00 -> 18.6 mm
- net Net-(D1-Pad1): track 18.5 -> 0.00 mm
- net Net-(D8-Pad1): track 16.2 -> 0.00 mm
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Other:
- board text added: "Daylight on a stick by Blamm Daybreak Neo by Vector 3D V2.1"
- board text removed: "Daylight on a stick by Blamm Daybreak Neo by Vector 3D V2"

Commit message: Daylight (all) V2.2
The JST XH silkscreen did not match the connectors very well so it has been adjusted.
Added small front silkscreen to indicate pins
Adjusted one connector on day_mini that was misplaced 1mm.
Parts:
- J1, J2: footprint Connector_JST:JST_XH_S3B-XH-A_1x03_P2.50mm_Horizontal -> Daylight:JST_XH_S3B-XH-A_1x03_P2.50mm_Horizontal Daylight
Other:
- board text added: "+ DO -"
- board text added: "- DI +"
- board text added: "Daylight on a stick by Blamm Daybreak Neo by Vector 3D V2.2"
- board text removed: "Daylight on a stick by Blamm Daybreak Neo by Vector 3D V2.1"

Commit message: Minor Updates
Parts:
- added G***: LOGO, LOGO, B.Cu at (203.1, 33.0)
Other:
- board text added: "Daylight on a stick by Blamm Daybreak Neo by Vector 3D V2.3"
- board text removed: "Daylight on a stick by Blamm Daybreak Neo by Vector 3D V2.2"

Commit message: Minor LED Updates
Parts:
- added REF**: Tab, kikit:Tab, F.Cu at (120.0, 38.5)
- added REF**: Tab, kikit:Tab, F.Cu at (251.0, 27.5)
- added REF**: Tab, kikit:Tab, F.Cu at (120.0, 27.5)
- added REF**: Tab, kikit:Tab, F.Cu at (45.0, 38.5)
- added REF**: Tab, kikit:Tab, F.Cu at (251.0, 38.5)
- added REF**: Tab, kikit:Tab, F.Cu at (193.5, 38.5)
- added REF**: Tab, kikit:Tab, F.Cu at (45.0, 27.5)
- added REF**: Tab, kikit:Tab, F.Cu at (193.5, 27.5)
Changed lines of the file:
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@@
       (net 14 "Net-(D10-Pad4)") (pinfunction "DOUT") (pintype "output"))
+  )
+  (footprint "kikit:Tab" (layer "F.Cu")
+    (at 120 38.5 90)
+    (descr "A symbol representing annotation for tab placement")
+    (attr exclude_from_pos_files exclude_from_bom)
+    (fp_text reference "REF**" (at 0 -2 90) (layer "F.SilkS") hide
+      (effects (font (size 1 1) (thickness 0.15)))
+    )
+    (fp_text value "Tab" (at -3 -1 90) (layer "Dwgs.User")
+      (effects (font (size 1.2 1.2) (thickness 0.2)))
+    )
+    (fp_text user "KIKIT: width: 8mm" (at -5.5 0) (layer "Dwgs.User")
+      (effects (font (size 1 1) (thickness 0.15)))
+    )
+    (fp_line (start 0.25 0) (end -0.75 -1) (layer "Dwgs.User") (width 0.3))
+    (fp_line (start 0.25 0) (end -2.75 0) (layer "Dwgs.User") (width 0.3))
+    (fp_line (start 0.25 1) (end 0.25 -1) (layer "Dwgs.User") (width 0.3))
+    (fp_line (start 0.25 0) (end -0.75 1) (layer "Dwgs.User") (width 0.3))
   )
   (footprint "Daylight:XL-3528RGBW-WS2812B" (layer "F.Cu")
@@
       (net 5 "Net-(D1-Pad4)") (pinfunction "DOUT") (pintype "output"))
   )
+  (footprint "kikit:Tab" (layer "F.Cu")
+    (at 251 27.5 -90)
+    (descr "A symbol representing annotation for tab placement")
+    (attr exclude_from_pos_files exclude_from_bom)
+    (fp_text reference "REF**" (at 0 -2 90) (layer "F.SilkS") hide
+      (effects (font (size 1 1) (thickness 0.15)))
+    )
+    (fp_text value "Tab" (at -3 -1 90) (layer "Dwgs.User")
+      (effects (font (size 1.2 1.2) (thickness 0.2)))
+    )
+    (fp_text user "KIKIT: width: 8mm" (at -5.5 0) (layer "Dwgs.User")
+      (effects (font (size 1 1) (thickness 0.15)))
+    )
+    (fp_line (start 0.25 0) (end -2.75 0) (layer "Dwgs.User") (width 0.3))
+    (fp_line (start 0.25 0) (end -0.75 1) (layer "Dwgs.User") (width 0.3))
+    (fp_line (start 0.25 0) (end -0.75 -1) (layer "Dwgs.User") (width 0.3))
+    (fp_line (start 0.25 1) (end 0.25 -1) (layer "Dwgs.User") (width 0.3))
+  )
   (footprint "Daylight:XL-3528RGBW-WS2812B" (layer "F.Cu")
     (at 129 33 90)
@@
       (net 4 "Dend") (pinfunction "DOUT") (pintype "output"))
   )
+  (footprint "kikit:Tab" (layer "F.Cu")
+    (at 120 27.5 -90)
+    (descr "A symbol representing annotation for tab placement")
+    (attr exclude_from_pos_files exclude_from_bom)
+    (fp_text reference "REF**" (at 0 -2 90) (layer "F.SilkS") hide
+      (effects (font (size 1 1) (thickness 0.15)))
+    )
+    (fp_text value "Tab" (at -3 -1 90) (layer "Dwgs.User")
+      (effects (font (size 1.2 1.2) (thickness 0.2)))
+    )
+    (fp_text user "KIKIT: width: 8mm" (at -5.5 0) (layer "Dwgs.User")
+      (effects (font (size 1 1) (thickness 0.15)))
+    )
+    (fp_line (start 0.25 0) (end -0.75 1) (layer "Dwgs.User") (width 0.3))
+    (fp_line (start 0.25 0) (end -0.75 -1) (layer "Dwgs.User") (width 0.3))
+    (fp_line (start 0.25 1) (end 0.25 -1) (layer "Dwgs.User") (width 0.3))
+    (fp_line (start 0.25 0) (end -2.75 0) (layer "Dwgs.User") (width 0.3))
+  )
   (footprint "Daylight:XL-3528RGBW-WS2812B" (layer "F.Cu")
     (at 148 33 90)
@@
     (pad "4" smd rect (at -1.35 0.75 90) (size 0.9 0.75) (layers "F.Cu" "F.Paste" "F.Mask")
       (net 6 "Net-(D2-Pad4)") (pinfunction "DOUT") (pintype "output"))
+  )
+  (footprint "kikit:Tab" (layer "F.Cu")
+    (at 45 38.5 90)
+    (descr "A symbol representing annotation for tab placement")
+    (attr exclude_from_pos_files exclude_from_bom)
+    (fp_text reference "REF**" (at 0 -2 90) (layer "F.SilkS") hide
+      (effects (font (size 1 1) (thickness 0.15)))
+    )
+    (fp_text value "Tab" (at -3 -1 90) (layer "Dwgs.User")
+      (effects (font (size 1.2 1.2) (thickness 0.2)))
+    )
+    (fp_text user "KIKIT: width: 8mm" (at -5.5 0) (layer "Dwgs.User")
+      (effects (font (size 1 1) (thickness 0.15)))
+    )
+    (fp_line (start 0.25 1) (end 0.25 -1) (layer "Dwgs.User") (width 0.3))
+    (fp_line (start 0.25 0) (end -0.75 1) (layer "Dwgs.User") (width 0.3))
+    (fp_line (start 0.25 0) (end -2.75 0) (layer "Dwgs.User") (width 0.3))
+    (fp_line (start 0.25 0) (end -0.75 -1) (layer "Dwgs.User") (width 0.3))
+  )
+  (footprint "kikit:Tab" (layer "F.Cu")
+    (at 251 38.5 90)
+    (descr "A symbol representing annotation for tab placement")
+    (attr exclude_from_pos_files exclude_from_bom)
+    (fp_text reference "REF**" (at 0 -2 90) (layer "F.SilkS") hide
+      (effects (font (size 1 1) (thickness 0.15)))
+    )
+    (fp_text value "Tab" (at -3 -1 90) (layer "Dwgs.User")
+      (effects (font (size 1.2 1.2) (thickness 0.2)))
+    )
+    (fp_text user "KIKIT: width: 8mm" (at -5.5 0) (layer "Dwgs.User")
+      (effects (font (size 1 1) (thickness 0.15)))
+    )
+    (fp_line (start 0.25 1) (end 0.25 -1) (layer "Dwgs.User") (width 0.3))
+    (fp_line (start 0.25 0) (end -0.75 -1) (layer "Dwgs.User") (width 0.3))
+    (fp_line (start 0.25 0) (end -0.75 1) (layer "Dwgs.User") (width 0.3))
+    (fp_line (start 0.25 0) (end -2.75 0) (layer "Dwgs.User") (width 0.3))
   )
   (footprint "Daylight:C_0805_2012Metric_Pad1.18x1.45mm_HandSolder_V3Dspec" (layer "F.Cu")
@@
     (pad "1" thru_hole circle locked (at 1.697056 1.697056) (size 0.8 0.8) (drill 0.5) (layers *.Cu *.Mask)
       (net 1 "GND") (pinfunction "1") (pintype "input"))
+  )
+  (footprint "kikit:Tab" (layer "F.Cu")
+    (at 193.5 38.5 90)
+    (descr "A symbol representing annotation for tab placement")
+    (attr exclude_from_pos_files exclude_from_bom)
+    (fp_text reference "REF**" (at 0 -2 90) (layer "F.SilkS") hide
+      (effects (font (size 1 1) (thickness 0.15)))
+    )
+    (fp_text value "Tab" (at -3 -1 90) (layer "Dwgs.User")
+      (effects (font (size 1.2 1.2) (thickness 0.2)))
+    )
+    (fp_text user "KIKIT: width: 8mm" (at -5.5 0) (layer "Dwgs.User")
+      (effects (font (size 1 1) (thickness 0.15)))
+    )
+    (fp_line (start 0.25 0) (end -0.75 -1) (layer "Dwgs.User") (width 0.3))
+    (fp_line (start 0.25 1) (end 0.25 -1) (layer "Dwgs.User") (width 0.3))
+    (fp_line (start 0.25 0) (end -0.75 1) (layer "Dwgs.User") (width 0.3))
+    (fp_line (start 0.25 0) (end -2.75 0) (layer "Dwgs.User") (width 0.3))
   )
   (footprint "Daylight:C_0805_2012Metric_Pad1.18x1.45mm_HandSolder_V3Dspec" (layer "F.Cu")
@@
     )
   )
+  (footprint "kikit:Tab" (layer "F.Cu")
+    (at 45 27.5 -90)
+    (descr "A symbol representing annotation for tab placement")
+    (attr exclude_from_pos_files exclude_from_bom)
+    (fp_text reference "REF**" (at 0 -2 90) (layer "F.SilkS") hide
+      (effects (font (size 1 1) (thickness 0.15)))
+    )
+    (fp_text value "Tab" (at -3 -1 90) (layer "Dwgs.User")
+      (effects (font (size 1.2 1.2) (thickness 0.2)))
+    )
+    (fp_text user "KIKIT: width: 8mm" (at -5.5 0) (layer "Dwgs.User")
+      (effects (font (size 1 1) (thickness 0.15)))
+    )
+    (fp_line (start 0.25 0) (end -0.75 -1) (layer "Dwgs.User") (width 0.3))
+    (fp_line (start 0.25 0) (end -2.75 0) (layer "Dwgs.User") (width 0.3))
+    (fp_line (start 0.25 1) (end 0.25 -1) (layer "Dwgs.User") (width 0.3))
+    (fp_line (start 0.25 0) (end -0.75 1) (layer "Dwgs.User") (width 0.3))
+  )
   (footprint "Daylight:C_0805_2012Metric_Pad1.18x1.45mm_HandSolder_V3Dspec" (layer "F.Cu")
     (at 95.2 33 90)
@@
     )
   )
+  (footprint "kikit:Tab" (layer "F.Cu")
+    (at 193.5 27.5 -90)
+    (descr "A symbol representing annotation for tab placement")
+    (attr exclude_from_pos_files exclude_from_bom)
+    (fp_text reference "REF**" (at 0 -2 90) (layer "F.SilkS") hide
+      (effects (font (size 1 1) (thickness 0.15)))
+    )
+    (fp_text value "Tab" (at -3 -1 90) (layer "Dwgs.User")
+      (effects (font (size 1.2 1.2) (thickness 0.2)))
+    )
+    (fp_text user "KIKIT: width: 8mm" (at -5.5 0) (layer "Dwgs.User")
+      (effects (font (size 1 1) (thickness 0.15)))
+    )
+    (fp_line (start 0.25 1) (end 0.25 -1) (layer "Dwgs.User") (width 0.3))
+    (fp_line (start 0.25 0) (end -2.75 0) (layer "Dwgs.User") (width 0.3))
+    (fp_line (start 0.25 0) (end -0.75 1) (layer "Dwgs.User") (width 0.3))
+    (fp_line (start 0.25 0) (end -0.75 -1) (layer "Dwgs.User") (width 0.3))
+  )
   (footprint "LOGO" (layer "B.Cu")
